File: OEP-2/OEP-2.sch (KiCad schematic (older format))
At the start: 24 parts

Commit message: подготовлена схема, определен габарит
Parts:
- added VT1: Транзистор_2Т3130А9, N_VD_HL:Транзистор_IRLML6344TR_SOT-23, symbol elements_2020:Транзистор_2Т3130А9
- added X1: Крепеж, N_X:Отверстие_М3, symbol elements_2020:Крепеж
- added XP1: Вилка_СНП346-7ВП21-1#0, symbol BIG_schemes:Вилка_СНП346-7ВП21-1#0
- added XP2: Вилка_СНП346-6ВП21-1#1N1N6, symbol BIG_schemes:Вилка_СНП346-6ВП21-1#1N1N6
- DD1: renamed from DD?; footprint (none) -> N_DD:Микросхема_5559ИНхх
- R7: renamed from R?; Номинал 240 Ом -> 1 кОм
- R8: renamed from R?; Номинал 100 кОм -> 1 кОм
- gave numbers to parts that had none: 21
Connections:
- net 5V: now also DD1.8 (Ucc), R8.1, XP1.4
- net EN-RS: now also DD1.2 (nRE), DD1.3 (DE), R8.2, VT1.3; no longer R7.1, R7.2, R8.1
- net GND: now also DD1.5 (GND), VT1.2, XP1.1, XP1.7; no longer R8.2
- net RS-A: now also DD1.6 (AY), XP2.2
- net RS-B: now also DD1.7 (BZ), XP2.3
- net RS-C: now also XP2.4
- net RX-MC: now also XP1.5
- net RX-RS: now also DD1.1 (RO)
- net SHLD: now also XP2.5
- net TX-MC: now also XP1.6
- net TX-RS: now also DD1.4 (DI)
- new net: R7.1, VT1.1
- new net EN-MC: R7.2, XP1.2, XP1.3
Other:
- moved on the sheet: C1, C2, C3, C4, C5, DD1, HL1, HL2, L1, L2, R1, R10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
