File: OEP-2/OEP-2.sch (KiCad schematic (older format))
At the start: 30 parts, among them X1 Крепеж

Commit message: назначены все посадочные места, готов сегмент  линий RS
Parts:
- added C6: Конденсатор_керамический, N_RLC:Конденсатор_SMD_IEC_0603, symbol OEP-2-rescue:Конденсатор_керамический-BIG_schemes
- C1, C3: footprint MOTOR_RLC:Конденсатор_SMD_IEC_0603 -> N_RLC:Конденсатор_SMD_IEC_0603; Номинал (none) -> 0,01u
- C2: footprint (none) -> Capacitor_Tantalum_SMD:CP_EIA-3528-21_Kemet-B_Pad1.50x2.35mm_HandSolder
- C4, C5: footprint MOTOR_RLC:Конденсатор_SMD_IEC_0603 -> N_RLC:Конденсатор_SMD_IEC_0603
- HL1, HL2: footprint MOTOR_VD_VT_HL:Светодиод_SMD_IEC_0603 -> N_VD_HL:Светодиод_SMD_IEC_0603
- VD1: footprint (none) -> N_VD_HL:Стабилитрон_корпус_КД-2_в_отверстие
- VD2, VD3: footprint (none) -> N_VD_HL:Стабилитрон_корпус_КД-2_в_отверстие; symbol OEP-2-rescue:Стабилитрон-BIG_schemes -> BIG_schemes:Стабилитрон
Connections:
- net 5V: now also C6.1
- net GND: now also C6.2
Changed lines of the file:
@@
 EESchema Schematic File Version 4
 LIBS:OEP-2-cache
-EELAYER 30 0
+EELAYER 29 0
 EELAYER END
 $Descr A2 23386 16535
@@
 F 0 "C1" V 15932 9591 138 0000 L CNB
 F 1 "Конденсатор_керамический" H 16100 9300 60  0001 C CNN
-F 2 "MOTOR_RLC:Конденсатор_SMD_IEC_0603" H 16000 9400 60  0001 C CNN
+F 2 "N_RLC:Конденсатор_SMD_IEC_0603" H 16000 9400 60  0001 C CNN
 F 3 "" H 16000 9400 60  0001 C CNN
 F 4 "0,01u" V 16167 9591 138 0000 L CNB "INFO"
+F 5 "0,01u" H 16000 9400 50  0001 C CNN "Номинал"
 	1    16000 9400
 	0    1    1    0
@@
 F 0 "C2" V 16932 9590 138 0000 L CNB
 F 1 "Конденсатор_электролитический" H 17100 9300 60  0001 C CNN
-F 2 "" H 17000 9400 60  0001 C CNN
+F 2 "Capacitor_Tantalum_SMD:CP_EIA-3528-21_Kemet-B_Pad1.50x2.35mm_HandSolder" H 17000 9400 60  0001 C CNN
 F 3 "" H 17000 9400 60  0001 C CNN
 F 4 "10u" V 17167 9590 138 0000 L CNB "INFO"
@@
 $EndComp
 $Comp
-L OEP-2-rescue:Стабилитрон-BIG_schemes VD3
+L BIG_schemes:Стабилитрон VD3
 U 1 1 60E0D466
 P 14500 3500
 F 0 "VD3" V 14700 4050 138 0000 R CNB
 F 1 "Стабилитрон_КС168В2" H 14600 3700 50  0001 C CNN
-F 2 "" H 14775 3500 50  0001 C CNN
+F 2 "N_VD_HL:Стабилитрон_корпус_КД-2_в_отверстие" H 14775 3500 50  0001 C CNN
 F 3 "" H 14775 3500 50  0001 C CNN
 F 4 "2.730" H 14600 3800 50  0001 C CNN "SYMBOL"
@@
 $EndComp
 $Comp
-L OEP-2-rescue:Стабилитрон-BIG_schemes VD2
+L BIG_schemes:Стабилитрон VD2
 U 1 1 60E0E58C
 P 14500 3200
 F 0 "VD2" V 14950 3000 138 0000 R CNB
 F 1 "Стабилитрон_КС168В2" H 14600 3400 50  0001 C CNN
-F 2 "" H 14775 3200 50  0001 C CNN
+F 2 "N_VD_HL:Стабилитрон_корпус_КД-2_в_отверстие" H 14775 3200 50  0001 C CNN
 F 3 "" H 14775 3200 50  0001 C CNN
 F 4 "2.730" H 14600 3500 50  0001 C CNN "SYMBOL"
@@
 F 0 "C3" V 15432 2991 138 0000 L CNB
 F 1 "Конденсатор_керамический" H 15600 2700 60  0001 C CNN
-F 2 "MOTOR_RLC:Конденсатор_SMD_IEC_0603" H 15500 2800 60  0001 C CNN
+F 2 "N_RLC:Конденсатор_SMD_IEC_0603" H 15500 2800 60  0001 C CNN
 F 3 "" H 15500 2800 60  0001 C CNN
 F 4 "0,01u" V 15667 2991 138 0000 L CNB "INFO"
+F 5 "0,01u" H 15500 2800 50  0001 C CNN "Номинал"
 	1    15500 2800
 	0    1    1    0
@@
 F 0 "VD1" V 18450 9600 138 0000 R CNB
 F 1 "Стабилитрон_КС168В2" H 18100 10000 50  0001 C CNN
-F 2 "" H 18275 9800 50  0001 C CNN
+F 2 "N_VD_HL:Стабилитрон_корпус_КД-2_в_отверстие" H 18275 9800 50  0001 C CNN
 F 3 "" H 18275 9800 50  0001 C CNN
 F 4 "2.730" H 18100 10100 50  0001 C CNN "SYMBOL"
@@
 F 0 "HL1" H 7334 2625 138 0000 L CNB
 F 1 "Светодиод" H 6600 2700 50  0001 C CNN
-F 2 "MOTOR_VD_VT_HL:Светодиод_SMD_IEC_0603" H 6775 2500 50  0001 C CNN
+F 2 "N_VD_HL:Светодиод_SMD_IEC_0603" H 6775 2500 50  0001 C CNN
 F 3 "" H 6775 2500 50  0001 C CNN
 F 4 "2.730" H 6600 2800 50  0001 C CNN "SYMBOL"
@@
 F 0 "HL2" H 7334 7625 138 0000 L CNB
 F 1 "Светодиод" H 6600 7700 50  0001 C CNN
-F 2 "MOTOR_VD_VT_HL:Светодиод_SMD_IEC_0603" H 6775 7500 50  0001 C CNN
+F 2 "N_VD_HL:Светодиод_SMD_IEC_0603" H 6775 7500 50  0001 C CNN
 F 3 "" H 6775 7500 50  0001 C CNN
 F 4 "2.730" H 6600 7800 50  0001 C CNN "SYMBOL"
@@
 F 0 "C4" V 16932 6791 138 0000 L CNB
 F 1 "Конденсатор_керамический" H 17100 6500 60  0001 C CNN
-F 2 "MOTOR_RLC:Конденсатор_SMD_IEC_0603" H 17000 6600 60  0001 C CNN
+F 2 "N_RLC:Конденсатор_SMD_IEC_0603" H 17000 6600 60  0001 C CNN
 F 3 "" H 17000 6600 60  0001 C CNN
 F 4 "0,01u" V 17167 6791 138 0000 L CNB "Номинал"
@@
 F 0 "C5" V 17932 6791 138 0000 L CNB
 F 1 "Конденсатор_керамический" H 18100 6500 60  0001 C CNN
-F 2 "MOTOR_RLC:Конденсатор_SMD_IEC_0603" H 18000 6600 60  0001 C CNN
+F 2 "N_RLC:Конденсатор_SMD_IEC_0603" H 18000 6600 60  0001 C CNN
 F 3 "" H 18000 6600 60  0001 C CNN
 F 4 "0,01u" V 18167 6791 138 0000 L CNB "Номинал"
@@
 Wire Wire Line
 	19000 2500 19900 2500
+$Comp
+L OEP-2-rescue:Конденсатор_керамический-BIG_schemes C6
+U 1 1 60E38AD8
+P 15000 9400
+F 0 "C6" V 14932 9591 138 0000 L CNB
+F 1 "Конденсатор_керамический" H 15100 9300 60  0001 C CNN
+F 2 "N_RLC:Конденсатор_SMD_IEC_0603" H 15000 9400 60  0001 C CNN
+F 3 "" H 15000 9400 60  0001 C CNN
+F 4 "0,01u" V 15167 9591 138 0000 L CNB "INFO"
+F 5 "0,01u" H 15000 9400 50  0001 C CNN "Номинал"
+	1    15000 9400
+	0    1    1    0
+$EndComp
+Wire Wire Line
+	16000 9000 15000 9000
+Wire Wire Line
+	15000 9000 15000 9300
+Connection ~ 16000 9000
+Wire Wire Line
+	16000 10000 15000 10000
+Wire Wire Line
+	15000 10000 15000 9600
 Wire Bus Line
 	4000 3600 4000 10500
@@
 Wire Bus Line
 	13500 2600 13500 10000
+Connection ~ 16000 10000
 $EndSCHEMATC
